File: hardware/battery_buddy-lite.kicad_sch (KiCad schematic)
At the start: 62 parts, among them J1 USB_C_Receptacle_USB2.0_16P, J2 BM04B-SRSS-TB, J3 Conn_01x10_MountingPin, J4 S4B-PH-SM4-TB, J5 Conn_01x01, SW1 SW_Push, U1 USBLC6-2P6, U2 LTC2959IDDB, U3 SN65HVD230DR, U4 ESP32-C3-MINI-1-N4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

Commit message: masking pin 11 of LTC2959
Parts:
- removed C21: 4.7uF 100V, Capacitor_SMD:C_2220_5750Metric, symbol Device:C
- removed C22: 100nF 100V, Capacitor_SMD:C_0603_1608Metric, symbol Device:C
- removed C23: 100nF, Capacitor_SMD:C_0402_1005Metric, symbol Device:C
- removed C24: 22uF 25V, Capacitor_SMD:C_1210_3225Metric, symbol Device:C
- removed L2: 56uH 2.0A, Inductor_SMD:L_Wuerth_HCI-1050, symbol Device:L_Ferrite
- removed R2: 100k, Resistor_SMD:R_0402_1005Metric, symbol Device:R
- removed R3: 7.15k, Resistor_SMD:R_0402_1005Metric, symbol Device:R
- removed U7: LMR51610XDBVR, Package_TO_SOT_SMD:SOT-23-6, symbol Regulator_Switching:LMR16006YQ
- C1, C2, C20, C3, C6, C8, C9: LCSC (none) -> C1525
- C10: value 47nF -> 4.7nF; LCSC (none) -> C53987
- C11, C15: LCSC (none) -> C55151
- C12: value 10uF -> 10uF 25V; LCSC (none) -> C13585
- C14, C7: value 10uF -> 10uF 6.3V; footprint Capacitor_SMD:C_1206_3216Metric -> Capacitor_SMD:C_0603_1608Metric; LCSC (none) -> C19702
- C17: footprint Capacitor_SMD:C_0805_2012Metric -> Capacitor_SMD:C_0603_1608Metric; LCSC (none) -> C15849
- C18, C19: LCSC (none) -> C39148
- C25, C26: LCSC (none) -> C13585
- C27: LCSC (none) -> C1550
- C4: LCSC (none) -> C47339
- C5: LCSC (none) -> C52923
- D1, D2: value D_Schottky -> DSK14; footprint Diode_SMD:D_SOD-523 -> Diode_SMD:D_SOD-123F; LCSC (none) -> C7502711
- D3: value NUP2105L -> NUP2105LT1G; LCSC (none) -> C14486; Rotation Offset (none) -> 90
- J1: LCSC (none) -> C963411
- J2: value BM04B-SRSS-TB -> BM04B-SRSS-TB(LF)(SN); Rotation Offset (none) -> 180
- J3: value Conn_01x10_MountingPin -> S10B-PH-SM4-TB(LF)(SN); LCSC (none) -> C265014
- R1: value CSM2F-6918-L050J30 -> ARCS6918JL050A9; LCSC (none) -> C2979379
- R10, R11: LCSC (none) -> C23090
- R12: LCSC (none) -> C25745
- R13: LCSC (none) -> C25798
- R14, R7: LCSC (none) -> C25744
- R16: LCSC (none) -> C25769
- R4, R8, R9: LCSC (none) -> C25879
- R5, R6: LCSC (none) -> C25905
- SW1: value SW_Push -> SPST; footprint Button_Switch_SMD:SW_SPST_B3U-1000P -> Button_Switch_SMD:SW_Push_SPST_NO_Alps_SKRK; LCSC (none) -> C720477; MPN (none) -> TS-1088-AR02016
- U1: Rotation Offset (none) -> 180
Connections:
- net CAN_RX is gone; now on net CAN_2_MCU: U4.20 (GPIO6)
- net CAN_TX is gone; now on net MCU_2_CAN: U4.21 (GPIO7)
- no-connect marks 8 -> 7
Other:
- note added: "+12V ±5% 250mA"
- note added: "+3.3V ±2.5% 500mA"
- note added: "ESP32-C3-MINI-1"
- note added: "I_{q} = 20uA Eff = ?%"
- note added: "I_{q} = ?uA Eff = ?%"
- note added: "Need to sort out these pins"
- note added: "This has a high quiecent. Find something better?"
- note added: "U4 → offset 'up' ? J2 → Maybe also make right angle? R1 → flip to bottom U5 → fix/finish footprint USB C is 'difficlult'"
- note removed: "ESP32"
- note removed: "How about TPSM365R6RDNR?"
- note removed: "I_{q} = 20uA"
- note removed: "Replace with ASR-M-7-0.25F Or even CSM2F-6918-L050J30"
- note removed: "TVS diode for VDD? SMAJ58A is a little too large. Max battery will be 50.5V But regen may take it higher Will have an active resistor clamp, but how well will that work? LTC2959 Abs Max is 65V SMAJ51A is 51.0 V_{r}, 56.7 V_{br min}, 62.70 V_{br max}"
- moved on the sheet: C10, C11, C12, C13, C14, C15, C16, C17, C2, C25, C26, C27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

Commit message: updating board shape and USB C conn
Parts:
- J1: LCSC C963411 -> C393939
Other:
- note added: "Turns out this has pretty terrible light load efficiencies. May need to rethink this regulator"
- note added: "U4 → offset 'up' ? J2 → Maybe also make right angle? U5 → fix/finish footprint"
- note removed: "U4 → offset 'up' ? J2 → Maybe also make right angle? R1 → flip to bottom U5 → fix/finish footprint USB C is 'difficlult'"
Changed lines of the file:
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@@
 		)
 	)
+	(text "Need to sort out these pins"
+		(exclude_from_sim no)
+		(at 228.6 187.452 0)
+		(effects
+			(font
+				(size 1.27 1.27)
+				(color 255 0 0 1)
+			)
+			(justify left bottom)
+		)
+	)
 	(text "+3.3V ±2.5%\n500mA"
 		(exclude_from_sim no)
@@
 	(text "Need to sort out these pins"
 		(exclude_from_sim no)
-		(at 239.268 168.91 0)
+		(at 228.346 167.386 0)
 		(effects
 			(font
@@
 				(color 255 0 0 1)
 			)
-			(justify left)
+			(justify left bottom)
 		)
 	)
-	(text "U4 → offset 'up' ?\nJ2 → Maybe also make right angle?\nR1 → flip to bottom\nU5 → fix/finish footprint\nUSB C is 'difficlult'"
+	(text "U4 → offset 'up' ?\nJ2 → Maybe also make right angle?\nU5 → fix/finish footprint"
 		(exclude_from_sim no)
 		(at 431.292 141.478 0)
@@
 		)
 	)
+	(text "Need to sort out these pins"
+		(exclude_from_sim no)
+		(at 228.6 172.466 0)
+		(effects
+			(font
+				(size 1.27 1.27)
+				(color 255 0 0 1)
+			)
+			(justify left bottom)
+		)
+	)
+	(text "Need to sort out these pins"
+		(exclude_from_sim no)
+		(at 147.574 149.606 0)
+		(effects
+			(font
+				(size 1.27 1.27)
+				(color 255 0 0 1)
+			)
+			(justify right bottom)
+		)
+	)
 	(text "External\nCAN Bus\nConnector"
 		(exclude_from_sim no)
@@
 		)
 	)
+	(text "Need to sort out these pins"
+		(exclude_from_sim no)
+		(at 229.108 182.372 0)
+		(effects
+			(font
+				(size 1.27 1.27)
+				(color 255 0 0 1)
+			)
+			(justify left bottom)
+		)
+	)
+	(text "Need to sort out these pins"
+		(exclude_from_sim no)
+		(at 228.854 174.752 0)
+		(effects
+			(font
+				(size 1.27 1.27)
+				(color 255 0 0 1)
+			)
+			(justify left bottom)
+		)
+	)
 	(text "VESC Express\ncompatible"
 		(exclude_from_sim no)
@@
 		)
 	)
+	(text "Turns out this has pretty terrible light load efficiencies.\nMay need to rethink this regulator"
+		(exclude_from_sim no)
+		(at 62.23 272.288 0)
+		(effects
+			(font
+				(size 1.27 1.27)
+				(color 255 0 0 1)
+			)
+			(justify left bottom)
+		)
+	)
+	(text "Need to sort out these pins"
+		(exclude_from_sim no)
+		(at 228.854 184.658 0)
+		(effects
+			(font
+				(size 1.27 1.27)
+				(color 255 0 0 1)
+			)
+			(justify left bottom)
+		)
+	)
 	(text "I_{q} = 20uA\nEff = ?%"
 		(exclude_from_sim no)
@@
 		)
 	)
+	(text "Need to sort out these pins"
+		(exclude_from_sim no)
+		(at 147.574 147.066 0)
+		(effects
+			(font
+				(size 1.27 1.27)
+				(color 255 0 0 1)
+			)
+			(justify right bottom)
+		)
+	)
 	(junction
 		(at 189.23 115.57)
@@
 			)
 		)
-		(property "LCSC" "C963411"
+		(property "LCSC" "C393939"
 			(at 388.62 53.34 0)
 			(effects
